Commit message: 2dof vehicle without hydro

File: URDFs/alpha_seabotix_virtualmasses.urdf (robot description, URDF)
Before this commit: robot uvms_alpha_seabotix, 30 links, 29 joints
Links:
- removed link virtual_x
- added link virtual_z, mass 18.0
Joints:
- removed joint x_prism
- removed joint y_prism
- added joint x_prismatic: type prismatic, parent virtual_z, child vehicle_base_link, origin xyz=0 0 0 rpy=0 0 0, axis 1.0 0.0 0.0
- added joint z_prismatic: type prismatic, parent base_link, child virtual_z, origin xyz=0 0 0 rpy=0 0 0
