Commit message: started integrating vehicle grav and buoy

File: URDFs/alpha_seabotix.urdf (robot description, URDF)
Before this commit: robot uvms_alpha_seabotix, 29 links, 28 joints
Links:
- link vehicle_base_link: mass None -> 22.2
Joints:
- joint vehicle_to_world: type fixed -> prismatic

Commit message: x y z and roll implemented

File: URDFs/alpha_seabotix.urdf (robot description, URDF)
Before this commit: robot uvms_alpha_seabotix, 30 links, 29 joints
Links:
- added link virtual_y, mass 0.
- added link virtual_z, mass 0.
Joints:
- added joint world_roll: type revolute, parent virtual_z, child vehicle_base_link, origin xyz=0 0 0 rpy=0 0 0, axis 1.0 0.0 0.0
- added joint z_prism: type prismatic, parent virtual_y, child virtual_z, origin xyz=0 0 0 rpy=0 0 0, axis 0.0 0.0 1.0
- joint y_prism: child vehicle_base_link -> virtual_y

Commit message: attempted pitch

File: URDFs/alpha_seabotix.urdf (robot description, URDF)
Before this commit: robot uvms_alpha_seabotix, 32 links, 31 joints
Links:
- added link virtual_roll, mass 0.
Joints:
- added joint world_pitch: type revolute, parent virtual_roll, child vehicle_base_link, origin xyz=0 0 0 rpy=0 0 0, axis 0.0 1.0 0.0
- joint world_roll: child vehicle_base_link -> virtual_roll
