Commit message: started Bravo URDF

File: URDFs/bravo_only.urdf (robot description, URDF)
Before this commit: robot bravo_7_example, 3 links, 2 joints
Links:
- added link bravo_1013_base_link; collision cylinder length=0.030 radius=0.046; collision cylinder length=0.1 radius=0.046
- added link bravo_1013_end_link; visual mesh filename=/home/hkolano/onr-dynamics-julia/bravo_meshes/RS2-1030.obj
- added link bravo_1013_joint_link; collision cylinder length=0.03 radius=0.046; visual mesh filename=/home/hkolano/onr-dynamics-julia/bravo_meshes/RS2-1013-end.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
- added link bravo_1023_0_base_link; collision cylinder length=0.03 radius=0.0408; collision cylinder length=0.0816 radius=0.0408
- added link bravo_1023_0_end_link
- added link bravo_1023_0_joint_link; collision cylinder length=0.080 radius=0.0408; visual mesh filename=/home/hkolano/onr-dynamics-julia/bravo_meshes/RS2-1023_0-en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
- added link bravo_1023_1_base_link
- added link bravo_1023_1_joint_link; collision cylinder length=0.0056 radius=0.0408; visual mesh filename=package://bpl_bravo_description/meshes/RS2-1023_1_end.stl
- added link bravo_1026_0_base_link; collision cylinder length=0.03 radius=0.0408; collision cylinder length=0.0816 radius=0.0408
- added link bravo_1026_0_end_link; visual mesh filename=/home/hkolano/onr-dynamics-julia/bravo_meshes/RS2-1026_1-en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
- added link bravo_1026_0_joint_link; collision cylinder length=0.080 radius=0.0408; visual mesh filename=/home/hkolano/onr-dynamics-julia/bravo_meshes/RS2-1026_0-en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
- added link bravo_1026_1_base_link
- added link bravo_1026_1_end_link
- added link bravo_1026_1_joint_link; visual cylinder length=0.0056 radius=0.0408; visual mesh filename=/home/hkolano/onr-dynamics-julia/bravo_meshes/RS2-1026_1-en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
Joints:
- added joint bravo_1013_end_joint: type fixed, parent bravo_1013_joint_link, child bravo_1013_end_link, origin xyz=0.046 0 -0.05055 rpy=3.14159 0 3.14159
- added joint bravo_1023_0_end_joint: type fixed, parent bravo_1023_0_joint_link, child bravo_1023_0_end_link, origin xyz=0.0408 0 -0.09385 rpy=3.14159 0 0
- added joint bravo_1026_0_end_joint: type fixed, parent bravo_1026_0_joint_link, child bravo_1026_0_end_link, origin xyz=0.0408 0 -0.09385 rpy=3.14159 0 0
- added joint bravo_1026_1_end_joint: type fixed, parent bravo_1026_1_joint_link, child bravo_1026_1_end_link, origin xyz=0 0 0.0056 rpy=0 0 3.14159
- added joint bravo_axis_b: type continuous, parent bravo_1023_1_base_link, child bravo_1023_1_joint_link, origin xyz=0 0 0.0005 rpy=0 0 0, axis 0 0 -1
- added joint bravo_axis_c: type revolute, parent bravo_1023_0_base_link, child bravo_1023_0_joint_link, origin xyz=0.042 0 0.0578 rpy=0 0 0, axis 0 -1 0, limit lower=0.0 upper=3.2 effort=0 velocity=0
- added joint bravo_axis_d: type revolute, parent bravo_1026_1_base_link, child bravo_1026_1_joint_link, origin xyz=0 0 0.0005 rpy=0 0 0, axis 0 0 -1, limit lower=0 upper=6.2 effort=0 velocity=0
- added joint bravo_axis_e: type revolute, parent bravo_1026_0_base_link, child bravo_1026_0_joint_link, origin xyz=0.042 0 0.0578 rpy=0 3.14 0, axis 0 -1 0, limit lower=0.0 upper=3.2 effort=0 velocity=0
- added joint bravo_axis_f: type revolute, parent bravo_1013_base_link, child bravo_1013_joint_link, origin xyz=0.046 0 0.0642 rpy=0 0 0, axis 0 -1 0, limit lower=0.0 upper=3.2 effort=0 velocity=0
- added joint bravo_b_base_joint: type fixed, parent bravo_1023_0_end_link, child bravo_1023_1_base_link, origin xyz=0 0 0 rpy=0 0 0
- added joint bravo_c_base_joint: type fixed, parent bravo_1026_1_end_link, child bravo_1023_0_base_link, origin xyz=0 0 0.0 rpy=0 0 0
- added joint bravo_d_base_joint: type fixed, parent bravo_1026_0_end_link, child bravo_1026_1_base_link, origin xyz=0 0 0 rpy=0 0 0
- added joint bravo_e_base_joint: type fixed, parent bravo_1013_end_link, child bravo_1026_0_base_link, origin xyz=0 0 0.182 rpy=0 0 0
- added joint bravo_f_base_joint: type fixed, parent bravo_1019_end_link, child bravo_1013_base_link, origin xyz=0 0 0 rpy=0 0 0

Commit message: fixed urdf except for jaws

File: URDFs/bravo_only.urdf (robot description, URDF)
Before this commit: robot bravo_7_example, 17 links, 16 joints
Links:
- added link bravo_1023_1_end_link
- added link bravo_1028_base_link; collision cylinder length=0.120 radius=0.0408; visual mesh filename=/home/hkolano/onr-dynamics-julia/bravo_meshes/RS2-1028.obj
- added link bravo_1028_end_link
- added link bravo_finger_jaws_base_link; collision cylinder length=0.02 radius=0.05; visual mesh filename=/home/hkolano/onr-dynamics-julia/bravo_meshes/RS2-257.obj
- added link bravo_finger_jaws_rs2_300_link; collision box size=0.14 0.04 0.045; visual mesh filename=/home/hkolano/onr-dynamics-julia/bravo_meshes/RS2-300.obj
- added link bravo_finger_jaws_rs2_301_link; collision box size=0.14 0.04 0.045; visual mesh filename=/home/hkolano/onr-dynamics-julia/bravo_meshes/RS2-301.obj
- added link bravo_jaws_base_link
- added link bravo_push_rod
- link bravo_1023_1_joint_link: geometry collision cylinder length=0.0056 radius=0.0408; visual mesh filename=/home/hkolano/onr-dynamics-julia/bravo_meshes/RS2-1023_1-en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
Joints:
- added joint bravo_1023_1_end_joint: type fixed, parent bravo_1023_1_joint_link, child bravo_1023_1_end_link, origin xyz=0 0 0.0056 rpy=0 0 0
- added joint bravo_1028_end_joint: type fixed, parent bravo_1028_base_link, child bravo_1028_end_link, origin xyz=0 0 0.120 rpy=-1.5707 -1.5707 0
- added joint bravo_a_base_joint: type fixed, parent bravo_1023_1_end_link, child bravo_1028_base_link, origin xyz=0 0 0 rpy=0 0 0
- added joint bravo_axis_a: type prismatic, parent bravo_jaws_base_link, child bravo_push_rod, origin xyz=0 0 0.009 rpy=0 0 0, axis 0 0 1, limit lower=0 upper=0.035 effort=10 velocity=10
- added joint bravo_finger_jaws_joint: type fixed, parent bravo_jaws_base_link, child bravo_finger_jaws_base_link, origin xyz=0 0 0 rpy=0 0 0
- added joint bravo_finger_jaws_rs2_300_joint: type revolute, parent bravo_finger_jaws_base_link, child bravo_finger_jaws_rs2_300_link, origin xyz=0.0097 -.033 0 rpy=1.5707 0 0, axis 0 0 -1, limit lower=0 upper=1.0 effort=10 velocity=10, mimic joint=bravo_axis_a multiplier=18 offset=0
- added joint bravo_finger_jaws_rs2_301_joint: type revolute, parent bravo_finger_jaws_base_link, child bravo_finger_jaws_rs2_301_link, origin xyz=0.0097 0.033 0 rpy=1.5707 0 0, axis 0 0 1, limit lower=0 upper=1.0 effort=10 velocity=10, mimic joint=bravo_finger_jaws_rs2_300_joint multiplier=1 offset=0
- added joint bravo_jaws_joint: type fixed, parent bravo_1028_end_link, child bravo_jaws_base_link, origin xyz= 0 0 0.0 rpy=0 0 0
- joint bravo_axis_e: origin xyz=0.042 0 0.0578 rpy=0 3.14 0 -> xyz=0.042 0 0.0578 rpy=0 0 0
