Commit message: some bravo testbed work; added added mass to sim_main_floating

File: URDFs/alpha_seabotix_nojoints.urdf (robot description, URDF)
Before this commit: robot uvms_alpha_seabotix, 28 links, 27 joints
Links:
- link vehicle_base_link: mass 22.2 -> 30.3

File: URDFs/bravo_testbed.urdf (robot description, URDF)
Before this commit: robot bravo_7_example, 25 links, 24 joints
Links:
- link bravo_push_rod: mass 5.0 -> None
